File: slices/[SLCa_SERV]_Servo_Motor_Controller/hardware/BREAD_Slice.kicad_pcb (KiCad board)
At the start: 2 copper layers, 70 x 100 mm, 16 parts, among them J1 Conn_01x10_Female, J2 Screw_Terminal_01x03, J3 Screw_Terminal_01x03, J4 Screw_Terminal_01x03, J5 Screw_Terminal_01x03, J6 Screw_Terminal_01x03, J7 Conn_01x03_Male, J8 Screw_Terminal_01x02

Commit message: restructuring for rpi boards
Other:
- net class Default removed
