File: slices/[SLCa_STEP]_Stepper_Motor_Controller/hardware/BREAD_Slice.kicad_sch (KiCad schematic)
At the start: 27 parts

Commit message: restructuring for rpi boards
Parts:
- A1, A2, A3, A4: value (none) -> Pololu_Breakout_A4988; footprint (none) -> Module:Pololu_Breakout-16_15.2x20.3mm
- C1, C2, C3: value (none) -> 10uF_t; footprint (none) -> OCI_UPL_FOOTPRINTS:C_2312
- D1, D2, D3, D4: value (none) -> 5V; footprint (none) -> Diode_SMD:D_1206_3216Metric_Pad1.42x1.75mm_HandSolder
- G1: value (none) -> Arduino_Nano_v3.x; footprint (none) -> Module:Arduino_Nano
- H1, H2, H3, H4: value (none) -> MountingHole; footprint (none) -> MountingHole:MountingHole_3.2mm_M3_DIN965_Pad
- J1: value (none) -> Conn_01x10_Female; footprint (none) -> Connector_PinSocket_2.54mm:PinSocket_1x10_P2.54mm_Horizontal
- J2: value (none) -> Screw_Terminal_01x04; footprint (none) -> TerminalBlock_TE-Connectivity:TerminalBlock_TE_282834-4_1x04_P2.54mm_Horizontal
- J3, J4: value (none) -> Screw_Terminal_01x08; footprint (none) -> TerminalBlock_TE-Connectivity:TerminalBlock_TE_282834-8_1x08_P2.54mm_Horizontal
- J5: value (none) -> Conn_01x03_Male; footprint (none) -> Connector_PinSocket_2.54mm:PinSocket_1x03_P2.54mm_Vertical
- J6: value (none) -> Screw_Terminal_01x02; footprint (none) -> TerminalBlock_TE-Connectivity:TerminalBlock_TE_282834-2_1x02_P2.54mm_Horizontal
- Logo1: value (none) -> Logo_Open_Hardware_Small; footprint (none) -> Symbol:OSHW-Symbol_6.7x6mm_SilkScreen
- R1, R2, R3, R4: value (none) -> 1k; footprint (none) -> Resistor_SMD:R_1206_3216Metric_Pad1.30x1.75mm_HandSolder
