File: slices/[SLCc_USBP]_USB_Port/hardware/BREAD_Slice.kicad_sch (KiCad schematic)
At the start: 19 parts

Commit message: restructuring for rpi boards
Parts:
- A1: value (none) -> Arduino_Nano_v3.x; footprint (none) -> Module:Arduino_Nano
- C1, C2: value (none) -> 10uF_t; footprint (none) -> OCI_UPL_FOOTPRINTS:C_2312
- C3: value (none) -> 10 nF; footprint (none) -> OCI_UPL_FOOTPRINTS:C_2312
- C4: value (none) -> 100 nF; footprint (none) -> Capacitor_SMD:C_1206_3216Metric_Pad1.33x1.80mm_HandSolder
- C5: value (none) -> 100nF_t; footprint (none) -> Capacitor_SMD:C_1206_3216Metric_Pad1.33x1.80mm_HandSolder
- FB1: value (none) -> Ferrite_Bead; footprint (none) -> OCI_UPL_FOOTPRINTS:R_1206_HandSoldering
- H1, H2, H3, H4: value (none) -> MountingHole; footprint (none) -> MountingHole:MountingHole_3.2mm_M3_DIN965_Pad
- J1: value (none) -> Conn_01x10_Female; footprint (none) -> Connector_PinSocket_2.54mm:PinSocket_1x10_P2.54mm_Horizontal
- J2, J3: value (none) -> USB_A; footprint (none) -> Connector_USB:USB_A_Molex_67643_Horizontal
- Logo1: value (none) -> Logo_Open_Hardware_Small; footprint (none) -> Symbol:OSHW-Symbol_6.7x6mm_SilkScreen
- R1: value (none) -> 10k; footprint (none) -> OCI_UPL_FOOTPRINTS:R_1206_HandSoldering
- R2: value (none) -> 1k; footprint (none) -> Resistor_SMD:R_1206_3216Metric_Pad1.30x1.75mm_HandSolder
- U1: value (none) -> FSUSB42MUX; footprint (none) -> Package_SO:MSOP-10_3x3mm_P0.5mm
- U2: value (none) -> FT232RL; footprint (none) -> Package_SO:SSOP-28_5.3x10.2mm_P0.65mm
