File: slices/[SLCi_HEAT]_Heating_Element_Controller/hardware/BREAD_Slice.kicad_pcb (KiCad board)
At the start: 2 copper layers, 70 x 100 mm, 21 parts, among them J1 Conn_01x10_Female, J2 Screw_Terminal_01x02, J3 Screw_Terminal_01x02, J4 Screw_Terminal_01x02, Q1 TIP120, Q2 TIP120, U1 MAX31855KASA

Commit message: restructuring for rpi boards
Other:
- net class Default removed
