File: slices/[SLCi_RLHT]_Relay_Heating_Element_Controller/hardware/BREAD_Slice.kicad_pcb (KiCad board)
At the start: 2 copper layers, 70 x 100 mm, 48 parts, among them J1 Conn_01x10_Female, J10 Term_PressFit_Phoenix_Contact, J11 Term_PressFit_Phoenix_Contact, J12 Term_PressFit_Phoenix_Contact, J13 Term_PressFit_Phoenix_Contact, J14 Term_PressFit_Phoenix_Contact, J15 Term_PressFit_Phoenix_Contact, J16 Term_PressFit_Phoenix_Contact, J17 Term_PressFit_Phoenix_Contact, J18 Term_PressFit_Phoenix_Contact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

Commit message: restructuring for rpi boards
Other:
- board text added: "LED"
- board text removed: "locked"
