File: slices/[SLCp_BUCK]_Buck_Converter_Signal_Generator/hardware/BREAD_Slice.kicad_pcb (KiCad board)
At the start: 2 copper layers, 70 x 100 mm, 17 parts, among them J1 Conn_01x10_Female, J2 Term_2, J3 Term_2, Q1 TIP120

Commit message: restructuring for rpi boards
Other:
- net class Default removed
