File: slices/[SLCp_SOLR]_Field_Solar_Power/hardware/BREAD_Slice.kicad_pcb (KiCad board)
At the start: 2 copper layers, 70 x 100 mm, 35 parts, among them J1 Conn_01x10_Female, J2 Screw_Terminal_01x02, J3 Screw_Terminal_01x02, U1 LM2576HVT-ADJ, U2 MCP73871

Commit message: restructuring for rpi boards
Other:
- net class Default removed
