File: slices/[SLCs_AAFT]_Audio_Analysis/hardware/BREAD_Slice.kicad_sch (KiCad schematic)
At the start: 53 parts

Commit message: restructuring for rpi boards
Parts:
- A1: value (none) -> Arduino_Nano_v3.x; footprint (none) -> Module:Arduino_Nano
- C1, C2: value (none) -> 10uF_t; footprint (none) -> OCI_UPL_FOOTPRINTS:C_2312
- C10, C11, C12, C4, C5, C6, C7, C8, C9: value (none) -> 0.1 uF; footprint (none) -> Capacitor_SMD:C_1206_3216Metric_Pad1.33x1.80mm_HandSolder
- C3: value (none) -> 10 uF; footprint (none) -> Capacitor_SMD:C_1206_3216Metric_Pad1.33x1.80mm_HandSolder
- H1, H2, H3, H4: value (none) -> MountingHole; footprint (none) -> MountingHole:MountingHole_3.2mm_M3_DIN965_Pad
- J1: value (none) -> Conn_01x10_Female; footprint (none) -> Connector_PinSocket_2.54mm:PinSocket_1x10_P2.54mm_Horizontal
- J2: value (none) -> Aux; footprint (none) -> Connector_Audio:Jack_3.5mm_CUI_SJ1-3533NG_Horizontal
- J3: value (none) -> Q_Inch; footprint (none) -> Connector_Audio:Jack_6.35mm_Neutrik_NMJ6HCD2_Horizontal
- Logo1: value (none) -> Logo_Open_Hardware_Small; footprint (none) -> Symbol:OSHW-Symbol_6.7x6mm_SilkScreen
- R1, R10, R11, R12, R2, R3, R4, R5, R6, R7, R8, R9: value (none) -> 1k; footprint (none) -> Resistor_SMD:R_1206_3216Metric_Pad1.30x1.75mm_HandSolder
- R13, R14, R15, R16: value (none) -> 500; footprint (none) -> Resistor_SMD:R_1206_3216Metric_Pad1.30x1.75mm_HandSolder
- R17: value (none) -> 400; footprint (none) -> Resistor_SMD:R_1206_3216Metric_Pad1.30x1.75mm_HandSolder
- R18, R19: value (none) -> 1.8 k; footprint (none) -> Resistor_SMD:R_1206_3216Metric_Pad1.30x1.75mm_HandSolder
- R20, R21: value (none) -> 900; footprint (none) -> Resistor_SMD:R_1206_3216Metric_Pad1.30x1.75mm_HandSolder
- R22, R23: value (none) -> 600; footprint (none) -> Resistor_SMD:R_1206_3216Metric_Pad1.30x1.75mm_HandSolder
- R24, R25: value (none) -> 450; footprint (none) -> Resistor_SMD:R_1206_3216Metric_Pad1.30x1.75mm_HandSolder
- R26: value (none) -> 360; footprint (none) -> Resistor_SMD:R_1206_3216Metric_Pad1.30x1.75mm_HandSolder
- RV1, RV2, RV3, RV4: value (none) -> 10k; footprint (none) -> Potentiometer_THT:Potentiometer_Bourns_3266W_Vertical
- U1, U2: value (none) -> MCP6004; footprint (none) -> Package_DIP:DIP-14_W7.62mm_Socket
