File: slices/[SLCs_CR10]_10A_Current_Sensor/hardware/BREAD_Slice.kicad_pcb (KiCad board)
At the start: 2 copper layers, 70 x 100 mm, 17 parts, among them J1 Conn_01x10_Female, J2 Screw_Terminal_01x02, J3 Screw_Terminal_01x02, J4 Screw_Terminal_01x02, J5 Screw_Terminal_01x02, U1 ACS723xMATR-10AB, U2 ACS723xMATR-10AB, U3 ACS723xMATR-10AB, U4 ACS723xMATR-10AB

Commit message: restructuring for rpi boards
Other:
- net class Default removed
