File: slices/[SLCs_CR20]_20A_Current_Sensor/hardware/BREAD_Slice.kicad_sch (KiCad schematic)
At the start: 21 parts

Commit message: restructuring for rpi boards
Parts:
- A1: value (none) -> Arduino_Nano_v3.x; footprint (none) -> Module:Arduino_Nano
- C1, C2: value (none) -> 10uF_t; footprint (none) -> OCI_UPL_FOOTPRINTS:C_2312
- H1, H2, H3, H4: value (none) -> MountingHole; footprint (none) -> MountingHole:MountingHole_3.2mm_M3_DIN965_Pad
- J1: value (none) -> Conn_01x10_Female; footprint (none) -> Connector_PinSocket_2.54mm:PinSocket_1x10_P2.54mm_Horizontal
- J2, J3, J4, J5, J6, J7, J8, J9: value (none) -> Conn_01x01_Male; footprint (none) -> Custom:Blade_Connector
- Logo1: value (none) -> Logo_Open_Hardware_Small; footprint (none) -> Symbol:OSHW-Symbol_6.7x6mm_SilkScreen
- U1, U2, U3, U4: value (none) -> ACS723xMATR-20AB; footprint (none) -> Package_SO:SOIC-16W_7.5x10.3mm_P1.27mm
