File: slices/[SLCs_THRM]_Thermocouple_Reader/hardware/BREAD_Slice.kicad_sch (KiCad schematic)
At the start: 34 parts

Commit message: restructuring for rpi boards
Parts:
- A1: value (none) -> Arduino_Nano_v3.x; footprint (none) -> Module:Arduino_Nano
- C1, C2: value (none) -> 10uF_t; footprint (none) -> OCI_UPL_FOOTPRINTS:C_2312
- C3, C4, C5, C6: value (none) -> 0.01 uF; footprint (none) -> Capacitor_SMD:C_1206_3216Metric_Pad1.33x1.80mm_HandSolder
- FB1, FB2, FB3, FB4, FB5, FB6, FB7, FB8: value (none) -> Ferrite_Bead_Small; footprint (none) -> Resistor_SMD:R_1206_3216Metric_Pad1.30x1.75mm_HandSolder
- H1, H2, H3, H4: value (none) -> MountingHole; footprint (none) -> MountingHole:MountingHole_3.2mm_M3_DIN965_Pad
- J1: value (none) -> Conn_01x10_Female; footprint (none) -> Connector_PinSocket_2.54mm:PinSocket_1x10_P2.54mm_Horizontal
- J2, J3, J4, J5: value (none) -> Screw_Terminal_01x02; footprint (none) -> TerminalBlock_TE-Connectivity:TerminalBlock_TE_282834-2_1x02_P2.54mm_Horizontal
- Logo1: value (none) -> Logo_Open_Hardware_Small; footprint (none) -> Symbol:OSHW-Symbol_6.7x6mm_SilkScreen
- R1, R2, R3, R4, R5: value (none) -> 10k; footprint (none) -> Resistor_SMD:R_1206_3216Metric_Pad1.30x1.75mm_HandSolder
- U1, U2, U3, U4: value (none) -> MAX31855KASA; footprint (none) -> Package_SO:SOIC-8_3.9x4.9mm_P1.27mm
