File: slices/[SLCs_PHDO]_pH_Dissolved_Oxygen_Sensor/hardware/RPi_Hat/RPi_Hat.kicad_pcb (KiCad board)
At the start: 2 copper layers, 65 x 56.5 mm, 5 parts, among them J2 RPi_GPIO

Commit message: Initial commit of discrete hbridge motor driver
Parts:
- added A1: Arduino_Nano_v3.x, Module:Arduino_Nano, F.Cu at (-14.8, 124.2)
- added A1: Arduino_Nano_v3.x, Module:Arduino_Nano, F.Cu at (194.6, 71.2)
- added C1: 10uF_t, Extras:C_1206_3216Metric_Pad1.33x1.80mm_HandSolder, B.Cu at (6.29, 125.3)
- added C2: 10uF_t, Extras:C_1206_3216Metric_Pad1.33x1.80mm_HandSolder, B.Cu at (-5.88, 133.6)
- added H1: MountingHole, MountingHole:MountingHole_3.2mm_M3_DIN965_Pad, F.Cu at (215.4, 70.2)
- added H10: MountingHole, MountingHole:MountingHole_3.2mm_M3_DIN965_Pad, F.Cu at (236.9, 70.2)
- added H11: MountingHole, MountingHole:MountingHole_3.2mm_M3_DIN965_Pad, F.Cu at (236.9, 77.4)
- added H12: MountingHole, MountingHole:MountingHole_3.2mm_M3_DIN965_Pad, F.Cu at (37.5, 69.0)
- added H12: MountingHole, MountingHole:MountingHole_3.2mm_M3_DIN965_Pad, F.Cu at (140.5, 107.5)
- added H2: MountingHole, MountingHole:MountingHole_3.2mm_M3_DIN965_Pad, F.Cu at (132.5, 107.5)
- added H2: MountingHole, MountingHole:MountingHole_3.2mm_M3_DIN965_Pad, F.Cu at (215.4, 77.4)
- added H3: MountingHole, MountingHole:MountingHole_3.2mm_M3_DIN965_Pad, F.Cu at (132.5, 74.5)
- added H3: MountingHole, MountingHole:MountingHole_3.2mm_M3_DIN965_Pad, F.Cu at (165.0, 73.5)
- added H4: MountingHole, MountingHole:MountingHole_3.2mm_M3_DIN965_Pad, F.Cu at (222.6, 70.2)
- added H4: MountingHole, MountingHole:MountingHole_3.2mm_M3_DIN965_Pad, F.Cu at (-22.6, 158.8)
- added H5: MountingHole, MountingHole:MountingHole_3.2mm_M3_DIN965_Pad, F.Cu at (222.6, 77.4)
- added H5: MountingHole, MountingHole:MountingHole_3.2mm_M3_DIN965_Pad, F.Cu at (108.4, 73.9)
- added H6: MountingHole, MountingHole:MountingHole_3.2mm_M3_DIN965_Pad, F.Cu at (141.5, 74.0)
- added H7: MountingHole, MountingHole:MountingHole_3.2mm_M3_DIN965_Pad, F.Cu at (229.8, 70.2)
- added H7: MountingHole, MountingHole:MountingHole_3.2mm_M3_DIN965_Pad, F.Cu at (108.4, 107.7)
- added H8: MountingHole, MountingHole:MountingHole_3.2mm_M3_DIN965_Pad, F.Cu at (229.8, 77.4)
- added H8: MountingHole, MountingHole:MountingHole_3.2mm_M3_DIN965_Pad, F.Cu at (-22.5, 69.0)
- added H9: MountingHole, MountingHole:MountingHole_3.2mm_M3_DIN965_Pad, F.Cu at (37.5, 159.0)
- added H9: MountingHole, MountingHole:MountingHole_3.2mm_M3_DIN965_Pad, F.Cu at (165.0, 107.5)
- added J2: Conn_01x05_Female, Connector_PinSocket_2.54mm:PinSocket_1x05_P2.54mm_Vertical, F.Cu at (125.8, 98.7)
- added J3: Conn_01x03_Male, Connector_PinSocket_2.54mm:PinSocket_1x03_P2.54mm_Vertical, F.Cu at (164.5, 157.4)
- added J4: Conn_01x03_Male, Connector_PinSocket_2.54mm:PinSocket_1x03_P2.54mm_Vertical, F.Cu at (34.5, 103.1)
- added J4: Conn_01x05_Female, Connector_PinSocket_2.54mm:PinSocket_1x05_P2.54mm_Vertical, F.Cu at (214.2, 100.1)
- added J5: Conn_01x03_Male, Connector_PinSocket_2.54mm:PinSocket_1x03_P2.54mm_Vertical, F.Cu at (218.8, 90.4)
- added J5: Conn_01x03_Male, Connector_PinSocket_2.54mm:PinSocket_1x03_P2.54mm_Vertical, F.Cu at (38.1, 103.1)
- added J6: Conn_01x05_Female, Connector_PinSocket_2.54mm:PinSocket_1x05_P2.54mm_Vertical, F.Cu at (158.0, 96.5)
- added J6: Conn_01x03_Male, Connector_PinSocket_2.54mm:PinSocket_1x03_P2.54mm_Vertical, F.Cu at (11.5, 156.4)
- added J7: Conn_01x03_Male, Connector_PinSocket_2.54mm:PinSocket_1x03_P2.54mm_Vertical, F.Cu at (223.4, 90.4)
- added J7: Conn_01x03_Male, Connector_PinSocket_2.54mm:PinSocket_1x03_P2.54mm_Vertical, F.Cu at (11.5, 160.0)
- added J8: Conn_01x10_Female, Connector_PinSocket_2.54mm:PinSocket_1x10_P2.54mm_Horizontal, F.Cu at (-20.7, 102.9)
- added J8: Conn_01x03_Male, Connector_PinSocket_2.54mm:PinSocket_1x03_P2.54mm_Vertical, F.Cu at (228.0, 90.4)
- added Logo1: Logo_Open_Hardware_Small, Symbol:OSHW-Symbol_6.7x6mm_SilkScreen, F.Cu at (-13.4, 68.5)
Routing:
- net (no net): track 0.00 -> 934.7 mm, vias 0 -> 3
- net GND: track 0.00 -> 116.0 mm
- net +5V: track 0.00 -> 69.8 mm
- net +12V: track 0.00 -> 50.2 mm
- net /pH_DO/OFFpH: track 0.00 -> 42.8 mm
- net /pH_DO/TX2/SDA: track 0.00 -> 35.8 mm
- net /pH_DO/RX2/SCL: track 0.00 -> 29.7 mm
Other:
- board size 65 x 56.5 mm -> 196.1 x 102 mm
- board text added: "pH and Dissolved Oxygen SLC_PHDO R0 2022"
